File: PCB_868_Combined/S1G_Mod_868_CMB.sch (KiCad schematic (older format))
At the start: 42 parts, among them P1 CONN_02X06, T1 1909763-1, T2 1909763-1, U1 AP2112K-3.3TRG1, U2 ADF7023BCPZ, X1 ABS07-32.768KHZ-9-T, X2 FA-128_26.0000MF10Z-AC3

Commit message: PCB Created
PCB created and placemetn started. Going to be a more robust
implementatinn of XBee pro but bigger formfactor. going to require dual
antennas or external mixrer (perhaps another PCB "? )
Parts:
- P?: renamed from P1; footprint Pin_Headers:Pin_Header_Angled_2x06 -> (none)
- renumbered BL1 to BL?, C16 to C?, C18 to C?, C21 to C?, C12 to C?, C13 to C?, C19 to C?, C15 to C?, C14 to C?, C11 to C?, C6 to C?, C1 to C?, C17 to C?, C20 to C?, C10 to C?, C8 to C?, C9 to C?, C5 to C?, C7 to C?, C3 to C?, C4 to C?, C2 to C?, FB1 to FB?, L7 to L?, L6 to L?, L1 to L?, L3 to L?, L5 to L?, L2 to L?, L4 to L?, LED1 to LED?, R2 to R?, R4 to R?, R1 to R?, R3 to R?, T2 to T?, T1 to T?, U1 to U?, U2 to U?, X2 to X?, X1 to X?
