File: PCB_868_900_Separate/S1G_Mod_868.kicad_pcb (KiCad board)
At the start: 4 copper layers, 60 x 33.3 mm, 82 parts, among them J2 20021121-00010C4LF, J5 0475890001-MicroUSBPort, P1 61301621121, Q1 DMG2307L-7, SW1 CUS-12TB, SW2 B3U-1000P, T1 0732511150, T2 0732511150, U1 AP7361-33FGE-7, U2 ADF7023BCPZ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

Commit message: More LDO
LDO section on separate antenna version retooled to be more like the
combined antenna version. Added additional fudicials on the bottom.
Parts:
- added FD4: FIDUCIAL, PCB_Footprints:FIDUCIAL, B.Cu at (115.2, 60.7)
- added FD5: FIDUCIAL, PCB_Footprints:FIDUCIAL, B.Cu at (57.8, 36.2)
- added FD6: FIDUCIAL, PCB_Footprints:FIDUCIAL, B.Cu at (57.8, 60.7)
- moved LED4 7.62 mm to (105.8, 47.1), turned to 180 degrees
- moved R10 6.53 mm to (107.9, 47.1), turned to 0 degrees
- moved R1 0.92 mm to (106.5, 53.6)
- moved C6 0.92 mm to (107.3, 48.2)
- moved U1 0.92 mm to (107.0, 50.9)
- moved C1 0.75 mm to (108.1, 54.3)
- moved D1 0.56 mm to (110.3, 50.6)
- moved Q1 0.56 mm to (110.3, 53.4)
Routing:
- net (no net): track 9.83 -> 0.03 mm, vias 5 -> 1
- net GND: track 412.2 -> 408.5 mm, vias 162 -> 160
- net /ON_OFF: track 11.8 -> 11.2 mm
- net +3V3: track 23.7 -> 24.1 mm, vias 13 -> 12
